File: latton rt.kicad_pcb (KiCad board)
At the start: 2 copper layers, 74 x 44 mm, 38 parts, among them J1 Barrel_Jack, J2 Barrel_Jack, J3 5267-02A-X, J4 5267-02A-X, J5 XT60-M, SW1 SW_SPDT

Commit message: 2
Changed lines of the file:
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@@
       (outputformat 1)
       (mirror false)
-      (drillshape 1)
+      (drillshape 0)
       (scaleselection 1)
-      (outputdirectory "")
+      (outputdirectory "gerber/")
     )
   )
@@
     (fp_line (start -2.45 1.8) (end 3.95 1.8) (layer "F.Fab") (width 0.1))
     (fp_line (start 0 1.092893) (end 0.5 1.8) (layer "F.Fab") (width 0.1))
-    (pad "1" thru_hole roundrect (at 0 0) (size 1.7 1.85) (drill 0.85) (layers *.Cu *.Mask) (roundrect_rratio 0.147059)
+    (pad "1" thru_hole roundrect (at 0 0) (size 1.7 1.85) (drill 0.85) (layers *.Cu *.Mask) (roundrect_rratio 0.1470588235)
       (net 4 "Net-(J1-Pad2)") (pinfunction "1") (pintype "passive"))
     (pad "2" thru_hole oval (at 2.5 0) (size 1.7 1.85) (drill 0.85) (layers *.Cu *.Mask)
@@
     (fp_line (start 1 0.625) (end -1 0.625) (layer "F.Fab") (width 0.1))
     (fp_line (start -1 0.625) (end -1 -0.625) (layer "F.Fab") (width 0.1))
-    (pad "1" smd roundrect (at -0.9125 0 270) (size 1.025 1.4) (layers "F.Cu" "F.Paste" "F.Mask") (roundrect_rratio 0.243902)
+    (pad "1" smd roundrect (at -0.9125 0 270) (size 1.025 1.4) (layers "F.Cu" "F.Paste" "F.Mask") (roundrect_rratio 0.243902439)
       (net 3 "Net-(D1-Pad2)") (pintype "passive"))
-    (pad "2" smd roundrect (at 0.9125 0 270) (size 1.025 1.4) (layers "F.Cu" "F.Paste" "F.Mask") (roundrect_rratio 0.243902)
+    (pad "2" smd roundrect (at 0.9125 0 270) (size 1.025 1.4) (layers "F.Cu" "F.Paste" "F.Mask") (roundrect_rratio 0.243902439)
       (net 1 "Net-(J1-Pad1)") (pintype "passive"))
     (model "${KICAD6_3DMODEL_DIR}/Resistor_SMD.3dshapes/R_0805_2012Metric.wrl"
@@
     (fp_line (start 3.95 1.8) (end 4.95 0.8) (layer "F.Fab") (width 0.1))
     (fp_line (start 4.95 -3.1) (end -2.45 -3.1) (layer "F.Fab") (width 0.1))
-    (pad "1" thru_hole roundrect (at 0 0) (size 1.7 1.85) (drill 0.85) (layers *.Cu *.Mask) (roundrect_rratio 0.147059)
+    (pad "1" thru_hole roundrect (at 0 0) (size 1.7 1.85) (drill 0.85) (layers *.Cu *.Mask) (roundrect_rratio 0.1470588235)
       (net 4 "Net-(J1-Pad2)") (pinfunction "1") (pintype "passive"))
     (pad "2" thru_hole oval (at 2.5 0) (size 1.7 1.85) (drill 0.85) (layers *.Cu *.Mask)
