File: latton rt.kicad_sch (KiCad schematic)
At the start: 8 parts, among them J1 Barrel_Jack, J2 Barrel_Jack, J3 5267-02A-X, J4 5267-02A-X, J5 XT60-M, SW1 SW_SPDT

Commit message: 2
Parts:
- D1: LCSC Part # (none) -> C2286
- R1: LCSC Part # (none) -> C17617
Changed lines of the file:
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@@
+      (effects (font (size 1.27 1.27)) hide)
+    )
+    (property "LCSC Part #" "C2286" (id 4) (at 129.54 55.88 0)
       (effects (font (size 1.27 1.27)) hide)
     )
@@
       (effects (font (size 1.27 1.27)) hide)
     )
+    (property "LCSC Part #" "C17617" (id 4) (at 139.7 55.88 0)
+      (effects (font (size 1.27 1.27)) hide)
+    )
